File: SEQ/minuterie556/minuterie556.kicad_pcb (KiCad board)
At the start: 2 copper layers, 17 parts, among them J1 Conn_01x02_Pin, J2 Barrel_Jack, J3 Conn_01x04_Pin, K1 SANYOU_SRD_Form_C, U3 LM556

Commit message: disposition en rectangle
Parts:
- moved J2 89.1 mm to (63.5, 68.6)
- moved J3 82.6 mm to (71.2, 68.6), turned to 0 degrees
- moved K1 82.1 mm to (48.9, 79.7), turned to 0 degrees
- moved D2 79.9 mm to (53.3, 88.9), turned to 0 degrees
- moved J1 79.7 mm to (50.8, 68.6), turned to 0 degrees
- moved D4 75.0 mm to (58.4, 114.3)
- moved D3 73.4 mm to (76.2, 91.4)
- moved C3 71.5 mm to (63.5, 111.8), turned to 0 degrees
- moved R3 66.5 mm to (71.1, 106.7), turned to 180 degrees
- moved D1 64.2 mm to (58.4, 91.4), turned to 180 degrees
- moved C2 59.9 mm to (71.1, 114.3)
- moved R2 55.9 mm to (76.2, 99.1), turned to -90 degrees
- moved BZ1 55.4 mm to (64.8, 121.9), turned to 180 degrees
- moved RV1 55.1 mm to (71.1, 76.2), turned to 180 degrees
- moved C1 53.0 mm to (71.2, 83.8)
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Routing:
- net Net-(D1-K): track 78.3 -> 10.4 mm
- net GNDREF: track 86.4 -> 136.7 mm
- net Net-(D2-A): track 52.6 -> 7.62 mm
- net Net-(D3-K): track 22.5 -> 61.6 mm
- net VCC: track 33.6 -> 65.9 mm
- net Net-(U3B-THR): track 58.6 -> 33.3 mm
- net Net-(D3-A): track 5.12 -> 27.1 mm
- net Net-(U3B-CV): track 34.3 -> 14.0 mm
- net Net-(U3A-THR): track 11.7 -> 25.0 mm
- net Net-(D4-A): track 11.5 -> 2.54 mm
- net +12C: track 6.80 -> 13.2 mm
- net Net-(BZ1--): track 10.7 -> 12.5 mm
- net GND1: track 22.4 -> 21.1 mm
- net Net-(U3B-DIS): track 8.89 -> 9.72 mm
